File: DenkyD4.sch (EAGLE design)
At the start: 41 parts, among them J1 CON_HEADER_1X06NO_SILK, J2 CON_HEADER_1X06NO_SILK, Q1 MUN5214DW1T1G, Q2 BSS138, SW1 RESET, U1 ESP32-PICO-D4, U2 FT231XQ-R, U3 AP2112K

Commit message: Updated to V1.2
Parts:
- removed C10: 100nF, _c2h:CAP0402-CAP-OK
- removed E1: NN03-320, _c2h:NN03-320
- removed R10, R11: 0R, _c2h:RESISTOR0603-RES
- removed RB, RG: 150, _c2h:RESISTOR0402-RES
- removed RGB: ASMB-KTF0-0A306, Particle:RGB-LED-CLMVB-FKARGB
- removed RR: 330, _c2h:RESISTOR0402-RES
- removed TINFO: 1X2-3.5MM, adafruit:1X2-3.5MM
- removed UFL: U.FL-R-SMT-1, Kris:U.FL-R-SMT-1
- removed USB: ZX62-B-5PA, Seeed-Connector:MICRO-USB-SMD(ZX62-B-5PA)
- added ANT: NN01-102, _c2h:NN01-102320
- added D1: 1N4148, microbuilder:DIODESOD-523
- added J3: KF2EDGR-3.81-2P, _c2h:1X2-3.5MM-3.5MM
- added LED: SK68051515, _c2h:SK68051515
- added LTIC: BLUE, OPL_Optoelectronics:SMD-LED-CLEAR-BLUE(0402)
- added Z1, Z3: 0R, _c2h:MATCHNET
- added Z2: DNP, _c2h:MATCHNET
- C3, C5: value 0.1uF -> 100nF
- C8, C9: value 47pF -> 100nF
- J1: value CON_HEADER_1X06NO_SILK -> US Type C; device _c2h:CON_HEADER_1X06NO_SILK -> SparkFun-Connectors:USB_C_4-LAYER-ISOLATED
- J2: value CON_HEADER_1X06NO_SILK -> Vertical Qwiic Connector; device _c2h:CON_HEADER_1X06NO_SILK -> _c2h:QWIIC_CONNECTOR
- Q2: device Seeed-Discrete:MOSFET-N-'' -> _c2h:SMD-MOSFET-N-CH-20V-2.1A-CJ2302(SOT-23)
- R3: value 220 -> 1K; device _c2h:RESISTOR0603-RES -> adafruit:TRIMPOTTC33X
- R5: value 10k -> 10K
- R7: value 100K -> 5.1K
- R8: value 27 -> 470; device _c2h:RESISTOR0402-RES -> LowPowerLab:RESISTOR0402-RES
- R9: value 27 -> 5.1K
- SW1: device Seeed-Switch:SMD-BUTTON(2P-3.0X2.5X1.2+0.4MM)-B3U-1000P-2P-SMD -> _c2h:SMD-BUTTON(2P-3.0X2.5X1.2+0.4MM)
- SW2: device microbuilder:SWITCH_TACT_SMT4.6X2.8 -> _c2h:SMD-BUTTON(2P-3.0X2.5X1.2+0.4MM)
- U2: value FT231XQ-R -> CH9106; device FT231XQ-R:FT231XQ-R -> microbuilder:CP2104
Connections:
- removed net ANT: R11.2, UFL.P$3
- removed net B$7: RB.2, RGB.2
- removed net DM: C9.1, R8.2, USB.D-
- removed net DP: C8.1, R9.2, USB.D+
- removed net G$6: RG.2, RGB.3
- removed net ID: R7.2, USB.ID
- removed net R$2: RGB.4, RR.2
- removed net VBUS: L1.1, USB.VBUS
- new net 5V: J1.VBUS, L1.1
- new net N$10: LTIC.+, R8.1
- new net N$11: J1.CC1, R9.2
- new net N$12: J1.CC2, R7.2
- new net N$6: U2G$1.RI
- new net N$8: C7.2, U2G$1.VDD, U2G$1.VIO
- new net VLED: C9.1, D1.C, LED.VDD
- net 3V3: now also J2.2, R8.2; no longer J1.5, J2.6, RGB.1, U2.VCCIO
- net D+: now also J1.D+, U2G$1.D+; no longer R8.1, U2.USBDM
- net D-: now also J1.D-, U2G$1.D-; no longer R9.1, U2.USBDP
- net DTR: now also U2G$1.DTR; no longer U2.DTR#
- net GND: now also J1.GND, J2.1, LED.VSS, R9.1, SW2.2, U2G$1.GND, U2G$2.TP, Z2.2; no longer C10.2, J1.6, SW2.P, SW2.P1, U2.GND, UFL.P$1, UFL.P$2, USB.GND
- net GPIO0: now also SW2.1; no longer SW2.S, SW2.S1
- net GPIO13: no longer J2.4
- net GPIO14: now also LED.DI
- net GPIO15: no longer J1.2
- net GPIO25: no longer RB.1
- net GPIO26: no longer RG.1
- net GPIO27: no longer RR.1
- net GPIO4: no longer J1.1
- net GPIO8: now also LTIC.-
- net LNA_IN: now also Z3.2; no longer R10.1, R11.1
- net N$1: now also Z1.1, Z2.1, Z3.1; no longer C10.1, U2.3V3OUT, U2.RESET#
- net N$13: now also ANT.1, Z1.2; no longer E1.FEED_BLUETOOTH, R10.2
- net N$3: now also R3.S; no longer R3.1
- net N$4: now also J3.1; no longer TINFO.1
- net N$5: now also J3.2, R3.A; no longer R3.2, TINFO.2
- net RESET: no longer J2.5
- net RTS: now also U2G$1.RTS; no longer U2.RTS#
- net RXD: now also U2G$1.TXD; no longer J2.2, U2.TXD
- net SCL: now also J2.4; no longer J1.3
- net SDA: now also J2.3; no longer J1.4
- net SHIELD: now also J1.SHLD; no longer USB.SHIELD
- net TXD: now also U2G$1.RXD; no longer J2.3, U2.RXD
- net V_USB: now also C8.1, D1.A, U2G$1.REGIN, U2G$1.VBUS; no longer C7.2, J2.1, U2.VCC
Other:
- note added: "CPU"
- note added: "I2C"
- note added: "Power Path"
- note added: "USB / Serial"
- note removed: "GPIO4"
- note removed: "GPIO5"
- note removed: "Headers"
- note removed: "USB TO SERIAL CONVERTER"
- moved on the sheet: C1, C2, C3, C4, C5, C6, C7, C8, C9, L1, L2, OK1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

Commit message: Bump to V1.2
Parts:
- added TGG, TP3, U$11, U$3, U$6: TP3, Particle:TP3
- J2: value Vertical Qwiic Connector -> Qwiic
Connections:
- removed net N$6: U2G$1.RI
- net 3V3: now also TP3.TP
- net GND: now also TGG.TP
- net GPIO25: now also U$11.TP
- net GPIO33: now also U$6.TP
- net GPIO7: now also U$3.TP
Other:
- note added: "I2C / GPIO"
- note removed: "I2C"
- moved on the sheet: J2, R1, R2

Commit message: Bump to V1.3a
Parts:
- added SLED: (no value), microbuilder:SOLDERJUMPER_CLOSED
- added TGG1, TGG2: TP3, Particle:TP3
Connections:
- new net N$6: LTIC.-, SLED.2
- net GND: now also TGG1.TP
- net GPIO8: now also SLED.1; no longer LTIC.-
- net V_USB: now also TGG2.TP
Other:
- moved on the sheet: LTIC, R8
Changed lines of the file:
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@@
 <setting verticaltext="up"/>
 </settings>
-<grid distance="25" unitdist="mil" unit="mil" style="dots" multiple="1" display="yes" altdistance="5" altunitdist="mil" altunit="mil"/>
+<grid distance="0.1" unitdist="inch" unit="inch" style="lines" multiple="1" display="no" altdistance="0.01" altunitdist="inch" altunit="inch"/>
 <layers>
 <layer number="1" name="Top" color="4" fill="1" visible="no" active="no"/>
@@
 <part name="NAME" library="SparkFun-Aesthetics" deviceset="FRAME-A4L" device="" value="Value">
 <attribute name="CNAME" value="DenkyD4"/>
-<attribute name="CREVISION" value="1.2"/>
+<attribute name="CREVISION" value="1.3a"/>
 <attribute name="DESIGNER" value="Charles-Henri Hallard"/>
 </part>
@@
 <part name="U$3" library="Particle" deviceset="TP" device="3"/>
 <part name="GND13" library="supply1" deviceset="GND" device=""/>
+<part name="TGG1" library="Particle" deviceset="TP" device="3"/>
+<part name="TGG2" library="Particle" deviceset="TP" device="3"/>
+<part name="SLED" library="microbuilder" deviceset="SOLDERJUMPER_CLOSED" device=""/>
 </parts>
 <sheets>
@@
 <attribute name="VALUE" x="120.65" y="128.905" size="1.778" layer="96"/>
 </instance>
-<instance part="R8" gate="G$1" x="260.35" y="64.135" smashed="yes" rot="R90">
-<attribute name="NAME" x="258.8514" y="62.865" size="1.778" layer="95" rot="R90"/>
-<attribute name="VALUE" x="263.652" y="62.865" size="1.778" layer="96" rot="R90"/>
-</instance>
-<instance part="LTIC" gate="G$1" x="260.35" y="53.975" smashed="yes" rot="R270">
-<attribute name="NAME" x="265.43" y="55.88" size="1.27" layer="95" ratio="10" rot="R270"/>
-<attribute name="VALUE" x="255.27" y="56.515" size="1.27" layer="96" ratio="10" rot="R270"/>
+<instance part="R8" gate="G$1" x="255.905" y="69.85" smashed="yes" rot="R180">
+<attribute name="NAME" x="257.175" y="68.3514" size="1.778" layer="95" rot="R180"/>
+<attribute name="VALUE" x="257.175" y="73.152" size="1.778" layer="96" rot="R180"/>
+</instance>
+<instance part="LTIC" gate="G$1" x="261.62" y="63.5" smashed="yes" rot="R270">
+<attribute name="NAME" x="266.7" y="65.405" size="1.27" layer="95" ratio="10" rot="R270"/>
+<attribute name="VALUE" x="256.54" y="66.04" size="1.27" layer="96" ratio="10" rot="R270"/>
 </instance>
 <instance part="GND7" gate="1" x="25.4" y="125.095"/>
@@
 <instance part="U$6" gate="G$1" x="231.14" y="163.195"/>
 <instance part="U$11" gate="G$1" x="231.14" y="160.02"/>
-<instance part="U$16" gate="G$1" x="236.855" y="168.91" smashed="yes">
-<attribute name="VALUE" x="235.331" y="169.926" size="1.27" layer="96"/>
-</instance>
-<instance part="GND12" gate="1" x="236.22" y="151.765"/>
+<instance part="U$16" gate="G$1" x="244.475" y="168.91" smashed="yes">
+<attribute name="VALUE" x="242.951" y="169.926" size="1.27" layer="96"/>
+</instance>
+<instance part="GND12" gate="1" x="237.49" y="151.765"/>
 <instance part="U$3" gate="G$1" x="231.14" y="156.845"/>
 <instance part="GND13" gate="1" x="261.62" y="128.27"/>
+<instance part="TGG1" gate="G$1" x="231.14" y="151.765"/>
+<instance part="TGG2" gate="G$1" x="231.14" y="144.78"/>
+<instance part="SLED" gate="G$1" x="261.62" y="53.975" rot="R90"/>
 </instances>
 <busses>
@@
 <pinref part="TGG" gate="G$1" pin="TP"/>
 <pinref part="GND12" gate="1" pin="GND"/>
-<wire x1="236.22" y1="154.305" x2="233.68" y2="154.305" width="0.1524" layer="91"/>
+<wire x1="237.49" y1="154.305" x2="234.315" y2="154.305" width="0.1524" layer="91"/>
+<pinref part="TGG1" gate="G$1" pin="TP"/>
+<wire x1="234.315" y1="154.305" x2="233.68" y2="154.305" width="0.1524" layer="91"/>
+<wire x1="233.68" y1="151.765" x2="234.315" y2="151.765" width="0.1524" layer="91"/>
+<wire x1="234.315" y1="151.765" x2="234.315" y2="154.305" width="0.1524" layer="91"/>
+<junction x="234.315" y="154.305"/>
 </segment>
 </net>
@@
 <pinref part="R8" gate="G$1" pin="2"/>
 <wire x1="248.92" y1="69.85" x2="248.92" y2="71.755" width="0.1524" layer="91"/>
-<wire x1="260.35" y1="69.215" x2="260.35" y2="69.85" width="0.1524" layer="91"/>
-<wire x1="260.35" y1="69.85" x2="248.92" y2="69.85" width="0.1524" layer="91"/>
+<wire x1="250.825" y1="69.85" x2="248.92" y2="69.85" width="0.1524" layer="91"/>
 <pinref part="OK1" gate="G$1" pin="C"/>
 <wire x1="237.49" y1="48.895" x2="241.3" y2="48.895" width="0.1524" layer="91"/>
@@
 <pinref part="TP3" gate="G$1" pin="TP"/>
 <pinref part="U$16" gate="G$1" pin="3.3V"/>
-<wire x1="236.855" y1="166.37" x2="233.68" y2="166.37" width="0.1524" layer="91"/>
+<wire x1="244.475" y1="166.37" x2="233.68" y2="166.37" width="0.1524" layer="91"/>
 </segment>
 </net>
@@
 <segment>
 <pinref part="Q2" gate="G$1" pin="D"/>
-<wire x1="267.97" y1="48.895" x2="260.35" y2="48.895" width="0.1524" layer="91"/>
 <pinref part="R5" gate="G$1" pin="1"/>
 <junction x="248.92" y="48.895"/>
-<wire x1="260.35" y1="48.895" x2="248.92" y2="48.895" width="0.1524" layer="91"/>
+<wire x1="267.97" y1="48.895" x2="261.62" y2="48.895" width="0.1524" layer="91"/>
+<wire x1="261.62" y1="48.895" x2="248.92" y2="48.895" width="0.1524" layer="91"/>
 <wire x1="248.92" y1="48.895" x2="248.92" y2="50.165" width="0.1524" layer="91"/>
 <label x="267.97" y="48.895" size="1.27" layer="95" xref="yes"/>
-<pinref part="LTIC" gate="G$1" pin="-"/>
-<wire x1="260.35" y1="48.895" x2="260.35" y2="50.165" width="0.1524" layer="91"/>
-<junction x="260.35" y="48.895"/>
+<pinref part="SLED" gate="G$1" pin="1"/>
+<junction x="261.62" y="48.895"/>
 </segment>
 </net>
@@
 <wire x1="64.135" y1="144.78" x2="64.135" y2="142.24" width="0.1524" layer="91"/>
 </segment>
+<segment>
+<pinref part="TGG2" gate="G$1" pin="TP"/>
+<wire x1="233.68" y1="144.78" x2="236.22" y2="144.78" width="0.1524" layer="91"/>
+<label x="236.22" y="144.78" size="0.8128" layer="95" xref="yes"/>
+</segment>
 </net>
 <net name="GPIO26" class="0">
@@
 <segment>
 <pinref part="R8" gate="G$1" pin="1"/>
-<wire x1="260.35" y1="59.055" x2="260.35" y2="57.785" width="0.1524" layer="91"/>
+<wire x1="260.985" y1="69.85" x2="261.62" y2="69.85" width="0.1524" layer="91"/>
+<wire x1="261.62" y1="69.85" x2="261.62" y2="67.31" width="0.1524" layer="91"/>
 <pinref part="LTIC" gate="G$1" pin="+"/>
 </segment>
@@
 </segment>
 </net>
+<net name="N$6" class="0">
+<segment>
+<pinref part="LTIC" gate="G$1" pin="-"/>
+<pinref part="SLED" gate="G$1" pin="2"/>
+<wire x1="261.62" y1="59.055" x2="261.62" y2="59.69" width="0.1524" layer="91"/>
+</segment>
+</net>
